Commit message: cant add joint to skeleton / importing door as urdf robot

File: door_rot/hello.urdf (robot description, URDF)
Before this commit: robot myfirst, 2 links, 1 joints
Joints:
- joint base_to_door: origin xyz=0.00 0.0 0.0 -> xyz=0.4 -0.25 0.3

Commit message: -seg fault at sampling/solving, +motion kept together correctly

File: door_rot/hello.urdf (robot description, URDF)
Before this commit: robot myfirst, 2 links, 1 joints
Joints:
- joint base_to_door: limit lower=-1.57 upper=1.57 effort=0.32 velocity=1.57 -> lower=-3.17 upper=0.43 effort=0.05 velocity=1.57
