Commit message: FINDS SOLUTION for a given valid motion config as goal state + hello.urdf missing collision part added

File: door_rot/fetch.urdf (robot description, URDF)
Before this commit: robot fetch, 28 links, 27 joints
Links:
- removed link door_link
- link base_link: geometry collision mesh filename=file:///home/serboba/rb_ws/src/robowflex_resources/fetch/me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; visual mesh filename=file:///home/serboba/rb_ws/src/robowflex_resources/fetch/me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
- link bellows_link: geometry collision mesh filename=file:///home/serboba/rb_ws/src/robowflex_resources/fetch/me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; visual mesh filename=file:///home/serboba/rb_ws/src/robowflex_resources/fetch/me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
- link bellows_link2: geometry collision mesh filename=file:///home/serboba/rb_ws/src/robowflex_resources/fetch/me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; visual mesh filename=file:///home/serboba/rb_ws/src/robowflex_resources/fetch/me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
- link door: geometry collision box size=0.6 0.5 0.05; visual box size=0.6 0.5 0.05
- link elbow_flex_link: geometry collision mesh filename=file:///home/serboba/rb_ws/src/robowflex_resources/fetch/me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; visual mesh filename=file:///home/serboba/rb_ws/src/robowflex_resources/fetch/me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
- link estop_link: geometry collision mesh filename=file:///home/serboba/rb_ws/src/robowflex_resources/fetch/me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; visual mesh filename=file:///home/serboba/rb_ws/src/robowflex_resources/fetch/me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
- link forearm_roll_link: geometry collision mesh filename=file:///home/serboba/rb_ws/src/robowflex_resources/fetch/me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; visual mesh filename=file:///home/serboba/rb_ws/src/robowflex_resources/fetch/me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
- link gripper_link: geometry collision mesh filename=file:///home/serboba/rb_ws/src/robowflex_resources/fetch/me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; visual mesh filename=file:///home/serboba/rb_ws/src/robowflex_resources/fetch/me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
- link head_pan_link: geometry collision mesh filename=file:///home/serboba/rb_ws/src/robowflex_resources/fetch/me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; visual mesh filename=file:///home/serboba/rb_ws/src/robowflex_resources/fetch/me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
- link head_tilt_link: geometry collision mesh filename=file:///home/serboba/rb_ws/src/robowflex_resources/fetch/me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; visual mesh filename=file:///home/serboba/rb_ws/src/robowflex_resources/fetch/me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
- link l_gripper_finger_link: geometry collision mesh filename=file:///home/serboba/rb_ws/src/robowflex_resources/fetch/me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; visual mesh filename=file:///home/serboba/rb_ws/src/robowflex_resources/fetch/me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
- link l_wheel_link: geometry collision mesh filename=file:///home/serboba/rb_ws/src/robowflex_resources/fetch/me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; visual mesh filename=file:///home/serboba/rb_ws/src/robowflex_resources/fetch/me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
- link laser_link: geometry collision mesh filename=file:///home/serboba/rb_ws/src/robowflex_resources/fetch/me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; visual mesh filename=file:///home/serboba/rb_ws/src/robowflex_resources/fetch/me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
- link r_gripper_finger_link: geometry collision mesh filename=file:///home/serboba/rb_ws/src/robowflex_resources/fetch/me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; visual mesh filename=file:///home/serboba/rb_ws/src/robowflex_resources/fetch/me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
- link r_wheel_link: geometry collision mesh filename=file:///home/serboba/rb_ws/src/robowflex_resources/fetch/me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; visual mesh filename=file:///home/serboba/rb_ws/src/robowflex_resources/fetch/me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
- link shoulder_lift_link: geometry collision mesh filename=file:///home/serboba/rb_ws/src/robowflex_resources/fetch/me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; visual mesh filename=file:///home/serboba/rb_ws/src/robowflex_resources/fetch/me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
- link shoulder_pan_link: geometry collision mesh filename=file:///home/serboba/rb_ws/src/robowflex_resources/fetch/me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; visual mesh filename=file:///home/serboba/rb_ws/src/robowflex_resources/fetch/me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
- link torso_fixed_link: geometry collision mesh filename=file:///home/serboba/rb_ws/src/robowflex_resources/fetch/me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; visual mesh filename=file:///home/serboba/rb_ws/src/robowflex_resources/fetch/me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
- link torso_lift_link: geometry collision mesh filename=file:///home/serboba/rb_ws/src/robowflex_resources/fetch/me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; visual mesh filename=file:///home/serboba/rb_ws/src/robowflex_resources/fetch/me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
- link upperarm_roll_link: geometry collision mesh filename=file:///home/serboba/rb_ws/src/robowflex_resources/fetch/me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; visual mesh filename=file:///home/serboba/rb_ws/src/robowflex_resources/fetch/me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
- link wrist_flex_link: geometry collision mesh filename=file:///home/serboba/rb_ws/src/robowflex_resources/fetch/me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; visual mesh filename=file:///home/serboba/rb_ws/src/robowflex_resources/fetch/me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
- link wrist_roll_link: geometry collision mesh filename=file:///home/serboba/rb_ws/src/robowflex_resources/fetch/me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; visual mesh filename=file:///home/serboba/rb_ws/src/robowflex_resources/fetch/me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
Joints:
- removed joint door_link_base_joint
- joint base_to_door: limit lower=-1.57 upper=1.57 effort=0.32 velocity=1.57 -> lower=-3.17 upper=0.43 effort=0.05 velocity=1.57; origin xyz=0.00 0.0 0.0 -> xyz=0.40 -0.25 0.3; parent door_link -> base_link

File: door_rot/hello.urdf (robot description, URDF)
Before this commit: robot myfirst, 2 links, 1 joints
Links:
- removed link base_link1
- added link base_link
- link door: geometry collision box size=0.6 0.5 0.05; visual box size=0.6 0.5 0.05
Joints:
- joint base_to_door: limit lower=-3.17 upper=0.43 effort=0.05 velocity=1.57 -> lower=-1.60 upper=0.0 effort=0.05 velocity=1.57; parent base_link1 -> base_link

Commit message: robot moving on xyz axis + z rotation

File: door_rot/fetch.urdf (robot description, URDF)
Before this commit: robot fetch, 27 links, 26 joints
Links:
- removed link door
- added link move_x_axis
- added link move_y_axis
- added link pushgr
- added link rotate_z_axis
Joints:
- removed joint base_to_door
- added joint gripper_axis2: type continuous, parent wrist_roll_link, child pushgr, origin xyz=0.2 0 0 rpy=0 0 0, axis 1 0 0
- added joint move_x_axis_joint: type prismatic, parent move_x_axis, child move_y_axis, origin xyz=0 0 0 rpy=0 0 0, axis 1 0 0, limit lower=-0.5 upper=0.5 effort=10 velocity=20
- added joint move_y_axis_joint: type prismatic, parent move_y_axis, child rotate_z_axis, origin xyz=0 0 0 rpy=0 0 0, axis 0 1 0, limit lower=-0.5 upper=0.5 effort=10 velocity=20
- added joint rotate_z_joint: type revolute, parent rotate_z_axis, child base_link, origin xyz=0 0 0 rpy=0 0 0, axis 0 0 1, limit lower=-3.14 upper=3.14 effort=10 velocity=20
