Commit message: now handling rotations included too, needs cleanup

File: door_rot/cube_scene.urdf (robot description, URDF)
Before this commit: robot cube_scene, 6 links, 5 joints
Joints:
- joint cube_joint: origin xyz=0.60 -0.2 0.84 rpy=0 0 0 -> xyz=1.60 -0.2 0.84 rpy=0 0 0
- joint door_joint1: axis 0.0 -1.0 0.0 -> 0 0 1; limit lower=0 upper=0.4 effort=0.05 velocity=1.57 -> lower=-1.60 upper=0 effort=0.05 velocity=1.57; type prismatic -> revolute
- joint door_joint2: origin xyz=0.6 -0.7 0.87 rpy=0 0 1.57 -> xyz=1.6 -0.7 0.87 rpy=0 0 1.57
