Commit message: quaternion calc fix, three doors sequence using rotation helper (no rot calculation needed), needs position simplification

File: door_rot/door_sequence/doors.urdf (robot description, URDF)
Before this commit: robot objects3, 4 links, 3 joints
Links:
- link door1: geometry collision box size=0.03 0.2 0.5; visual box size=0.03 0.2 0.5
- link door2: geometry collision box size=0.03 0.2 0.5; visual box size=0.03 0.2 0.5
- link door3: geometry collision box size=0.03 0.2 0.5; visual box size=0.03 0.2 0.5
Joints:
- joint base_to_door2: limit lower=0.0 upper=3.28 effort=0.05 velocity=1.57 -> lower=0.0 upper=2.00 effort=0.05 velocity=1.57; origin xyz=0.55 0.0 0.2 rpy=0 0 1.57 -> xyz=0.65 0.0 0.2 rpy=0 0 1.57
