Commit message: new iso-interpolation in isospace.cpp, bug: changing values at every iteration, interpolation buggy maybe

File: scripts/small_table_maze/maze.urdf (robot description, URDF)
Before this commit: robot cube_scene, 7 links, 6 joints
Joints:
- joint door_joint1: limit lower=-1.57 upper=1.57 effort=0.05 velocity=1.57 -> lower=-1.57 upper=0 effort=0.05 velocity=1.57
