Commit message: changing object structurefirst steps

File: scripts/envs/maze1.urdf (robot description, URDF)
Before this commit: robot maze1, 8 links, 7 joints
Links:
- removed link cube
- removed link door1
- removed link door2
- removed link door3
- added link cube_z
- added link link_0; collision box size=0.1 0.1 0.1; visual box size=0.1 0.1 0.1
- added link link_1; collision box size=0.03 0.5 0.173; visual box size=0.03 0.5 0.173
- added link link_2; collision box size=0.03 0.5 0.173; visual box size=0.03 0.5 0.173
- added link link_3; collision box size=0.03 0.45 0.173; visual box size=0.03 0.45 0.173
Joints:
- removed joint cube_joint
- removed joint cube_joint2
- removed joint door_joint1
- removed joint door_joint2
- removed joint door_joint3
- added joint link_0_joint_0: type prismatic, parent base_link, child cube_x, origin xyz=0.50 -0.8 0.75 rpy=0 0 0, axis 0 1 0, limit lower=0.0 upper=0.65 effort=0.05 velocity=1.57
- added joint link_0_joint_1: type prismatic, parent cube_x, child cube_z, origin xyz=0.0 0 0.0 rpy=0 0 0, axis 1 0 0, limit lower=-0.2 upper=0.7 effort=0.05 velocity=1.57
- added joint link_0_joint_2: type revolute, parent cube_z, child link_0, origin xyz=0.0 0 0.0 rpy=0 0 0, axis 0 0 1, limit lower=-1.57 upper=1.57 effort=0.05 velocity=1.57
- added joint link_1_joint_0: type revolute, parent base_link, child link_1, origin xyz=0.75 -1.125 0.755 rpy=0 0 0, axis 0 0 1, limit lower=-1.57 upper=1.57 effort=5 velocity=1.57
- added joint link_2_joint_0: type revolute, parent base_link, child link_2, origin xyz=1.25 -0.575 0.755 rpy=0 0 -1.57, axis 0 0 1, limit lower=-1.57 upper=1.57 effort=5 velocity=1.57
- added joint link_3_joint_0: type revolute, parent base_link, child link_3, origin xyz=0.75 -0.525 0.755 rpy=0 0 0, axis 0.0 0.0 1, limit lower=-1.57 upper=1.57 effort=5 velocity=1.57
- joint goal: axis 0 1 0 -> (none)
- joint table_j: axis 0 1 0 -> (none)

File: scripts/envs/maze2.urdf (robot description, URDF)
Before this commit: robot maze2, 9 links, 8 joints
Links:
- removed link cube
- removed link door1
- removed link door2
- removed link obs
- added link cube_z
- added link link_0; collision box size=0.1 0.1 0.1; visual box size=0.1 0.1 0.1
- added link link_1; collision box size=0.05 0.33 0.16; visual box size=0.05 0.33 0.16
- added link link_2; collision box size=0.1 0.25 0.1; visual box size=0.1 0.25 0.1
- added link link_t; visual box size=0.05 0.035 0.025
- added link obs_z
Joints:
- removed joint cube_joint
- removed joint cube_joint2
- removed joint door_joint1
- removed joint obs_joint
- removed joint obs_joint2
- added joint link_0_joint_0: type prismatic, parent base_link, child cube_x, origin xyz=0.30 -0.8 0.87 rpy=0 0 0, axis 1 0 0, limit lower=-0.1 upper=0.85 effort=0.05 velocity=1.57
- added joint link_0_joint_1: type prismatic, parent cube_x, child cube_z, origin xyz=0.0 0 0.0 rpy=0 0 0, axis 0 1 0, limit lower=0.0 upper=1.05 effort=0.05 velocity=1.57
- added joint link_0_joint_2: type revolute, parent cube_z, child link_0, origin xyz=0.0 0 0.0 rpy=0 0 0, axis 0 0 1, limit lower=-1.57 upper=1.57 effort=0.05 velocity=1.57
- added joint link_1_joint_0: type prismatic, parent base_link, child link_1, origin xyz=0.45 -0.735 0.89 rpy=0 0 0, axis 1 0 0, limit lower=-0.25 upper=0.5 effort=5 velocity=1.57
- added joint link_2_joint_0: type prismatic, parent base_link, child obs_x, origin xyz=0.95 -0.75 0.87 rpy=0 0 0, axis 1 0 0, limit lower=-0.70 upper=0.20 effort=0.05 velocity=1.57
- added joint link_2_joint_1: type prismatic, parent obs_x, child obs_z, origin xyz=0.0 0 0.0 rpy=0 0 0, axis 0 1 0, limit lower=-0.1 upper=0.90 effort=0.05 velocity=1.57
- added joint link_2_joint_2: type revolute, parent obs_z, child link_2, origin xyz=0.0 0 0.0 rpy=0 0 0, axis 0 0 1, limit lower=-1.57 upper=1.57 effort=0.05 velocity=1.57
- joint door_joint2: child door2 -> link_t; parent door1 -> link_1
- joint goal: origin xyz=1.02 -0.75 0.86 rpy=0 0 0 -> xyz=1.02 -0.75 0.87 rpy=0 0 0

File: scripts/envs/maze3.urdf (robot description, URDF)
Before this commit: robot maze3, 9 links, 8 joints
Links:
- removed link cube
- removed link door1
- removed link door2
- removed link door3
- removed link door4
- added link link_0; collision box size=0.1 0.1 0.1; visual box size=0.1 0.1 0.1
- added link link_1; collision box size=0.40 0.025 0.16; visual box size=0.40 0.025 0.16
- added link link_2; collision box size=0.40 0.025 0.16; visual box size=0.40 0.025 0.16
- added link link_3; collision box size=0.40 0.025 0.16; visual box size=0.40 0.025 0.16
- added link link_4; collision box size=0.40 0.025 0.16; visual box size=0.40 0.025 0.16
Joints:
- removed joint cube_joint
- removed joint cube_joint2
- removed joint door_joint1
- removed joint door_joint2
- removed joint door_joint3
- removed joint door_joint4
- added joint link_0_joint_0: type prismatic, parent base_link, child cube_x, origin xyz=0.40 -0.9 0.86 rpy=0 0 0, axis 1 0 0, limit lower=-0.17 upper=1.18 effort=0.05 velocity=1.57
- added joint link_0_joint_1: type prismatic, parent cube_x, child link_0, origin xyz=0.0 0 0.0 rpy=0 0 0, axis 0 1 0, limit lower=-0.1 upper=1.11 effort=0.05 velocity=1.57
- added joint link_1_joint_0: type prismatic, parent base_link, child link_1, origin xyz=0.39 -0.634 0.86 rpy=0 0 0, axis 1 0 0, limit lower=0 upper=1.02 effort=5 velocity=1.57
- added joint link_2_joint_0: type prismatic, parent base_link, child link_2, origin xyz=0.39 -0.166 0.86 rpy=0 0 0, axis 1 0 0, limit lower=0 upper=1.02 effort=5 velocity=1.57
- added joint link_3_joint_0: type prismatic, parent base_link, child link_3, origin xyz=1.41 -0.634 0.86 rpy=0 0 0, axis -1 0 0, limit lower=0 upper=1.02 effort=5 velocity=1.57
- added joint link_4_joint_0: type prismatic, parent base_link, child link_4, origin xyz=1.41 -0.166 0.86 rpy=0 0 0, axis -1 0 0, limit lower=0 upper=1.02 effort=5 velocity=1.57

File: scripts/envs/maze_vertical.urdf (robot description, URDF)
Before this commit: robot maze_vertical, 9 links, 8 joints
Links:
- removed link cube
- removed link door1
- removed link door2
- removed link door3
- removed link door4
- added link link_0; collision box size=0.1 0.1 0.1; visual box size=0.1 0.1 0.1
- added link link_1; collision box size=0.13 0.275 0.03; visual box size=0.13 0.275 0.03
- added link link_2; collision box size=0.13 0.03 0.21; visual box size=0.13 0.03 0.21
- added link link_3; collision box size=0.13 0.03 0.21; visual box size=0.13 0.03 0.21
- added link link_4; collision box size=0.13 0.21 0.03; visual box size=0.13 0.21 0.03
Joints:
- removed joint cube_joint
- removed joint cube_joint2
- removed joint door_joint1
- removed joint door_joint2
- removed joint door_joint3
- removed joint door_joint4
- added joint link_0_joint_0: type prismatic, parent base_link, child cube_x, origin xyz=0.75 0.1 1.3 rpy=0 0 0, axis 0 1 0, limit lower=-0.88 upper=0.08 effort=0.05 velocity=1.57
- added joint link_0_joint_1: type prismatic, parent cube_x, child link_0, origin xyz=0.0 0 0.0 rpy=0 0 0, axis 0 0 1, limit lower=-0.78 upper=0.1 effort=0.05 velocity=1.57
- added joint link_1_joint_0: type revolute, parent base_link, child link_1, origin xyz=0.745 0.2275 0.985 rpy=0 0 0, axis 1 0 0, limit lower=-1.57 upper=1.57 effort=0.05 velocity=1.57
- added joint link_2_joint_0: type revolute, parent base_link, child link_2, origin xyz=0.745 -0.075 0.74 rpy=0 0 0, axis 1 0 0, limit lower=-1.57 upper=1.57 effort=0.05 velocity=1.57
- added joint link_3_joint_0: type revolute, parent base_link, child link_3, origin xyz=0.745 -0.075 0.475 rpy=0 0 0, axis 1 0 0, limit lower=-1.57 upper=1.57 effort=0.05 velocity=1.57
- added joint link_4_joint_0: type revolute, parent base_link, child link_4, origin xyz=0.745 -0.325 1.29 rpy=0 0 0, axis 1 0 0, limit lower=-1.57 upper=0.00 effort=0.05 velocity=1.57

File: scripts/envs/simple_sliders.urdf (robot description, URDF)
Before this commit: robot simple_sliders, 4 links, 3 joints
Links:
- link base_link: mass None -> 0.001; geometry visual box size=0 0 0.2
- link link_0: mass None -> 0.001; geometry collision box size=0.2 0.2 1.6; visual box size=0.2 0.2 1.6
Joints:
- joint goal: origin xyz=0 -0.2 0.0 rpy=0 0 0 -> xyz=0 -1.0 0.2 rpy=1.5708 0 0
- joint link_0: axis 0 1 0 -> 0 0 1; limit lower=-1.0 upper=1.0 effort=0 velocity=0 -> lower=0 upper=1.0 effort=0 velocity=0; origin xyz=0 0.0 0.0 rpy=0 0 0 -> xyz=0 0 0.2 rpy=1.5708 0 0
- joint link_1: axis 0 0 1.0 -> 0 0 1
